File: KiCad Project/RB-Macro16.kicad_sch (KiCad schematic)
At the start: 67 parts, among them J1 USB_C_Receptacle, J2 AVR-ISP-6, SW1 SW_PUSH, U1 ATMEGA32U4, X1 XTAL_GND

Commit message: Placed ATMEGA
Placed ATMEGA and XTAL and caps and routed traces to them
Parts:
- added R5, R6: 22, Resistor_THT:R_Axial_DIN0207_L6.3mm_D2.5mm_P7.62mm_Horizontal, symbol Device:R
Connections:
- net col0: now also U1.31 (PC6); no longer U1.29 (PB5)
- net col2: now also U1.29 (PB5); no longer U1.31 (PC6)
- net col3: now also U1.28 (PB4); no longer U1.32 (PC7)
- net led0: now also U1.32 (PC7); no longer U1.28 (PB4)
- net rotA: now also U1.40 (PF1); no longer U1.37 (PF6)
- net rotB: now also U1.41 (PF0); no longer U1.36 (PF7)
- net row0: now also U1.36 (PF7); no longer U1.41 (PF0)
- net row1: now also U1.37 (PF6); no longer U1.40 (PF1)
- net row2: now also U1.38 (PF5); no longer U1.39 (PF4)
- net row3: now also U1.39 (PF4); no longer U1.38 (PF5)
- net at C18.1, X1.2: now also U1.16 (XTAL1); no longer U1.17 (XTAL2)
- net at C17.1, X1.1: now also U1.17 (XTAL2); no longer U1.16 (XTAL1)
- net at J1.A6 (D+), J1.B6 (D+): now also R6.1; no longer U1.4 (D+)
- net at J1.A7 (D-), J1.B7 (D-): now also R5.1; no longer U1.3 (D-)
- new net: R5.2, U1.3 (D-)
- new net: R6.2, U1.4 (D+)
Changed lines of the file:
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@@
   (junction (at 213.995 220.345) (diameter 0) (color 0 0 0 0)
   )
-  (junction (at 53.34 53.34) (diameter 0) (color 0 0 0 0)
-  )
   (junction (at 243.84 227.965) (diameter 0) (color 0 0 0 0)
   )
@@
   (junction (at 35.56 104.14) (diameter 0) (color 0 0 0 0)
   )
+  (junction (at 53.34 53.34) (diameter 0) (color 0 0 0 0)
+  )
   (junction (at 232.41 227.965) (diameter 0) (color 0 0 0 0)
   )
@@
   (junction (at 243.84 220.345) (diameter 0) (color 0 0 0 0)
   )
+  (junction (at 53.34 50.8) (diameter 0) (color 0 0 0 0)
+  )
   (junction (at 204.47 264.795) (diameter 0) (color 0 0 0 0)
   )
@@
   (junction (at 234.95 207.01) (diameter 0) (color 0 0 0 0)
   )
-  (junction (at 91.44 48.26) (diameter 0) (color 0 0 0 0)
-  )
   (junction (at 269.875 183.515) (diameter 0) (color 0 0 0 0)
   )
@@
   (junction (at 243.84 183.515) (diameter 0) (color 0 0 0 0)
   )
-  (junction (at 53.34 50.8) (diameter 0) (color 0 0 0 0)
-  )
   (junction (at 184.15 234.315) (diameter 0) (color 0 0 0 0)
   )
@@
   (junction (at 186.055 257.175) (diameter 0) (color 0 0 0 0)
   )
+  (junction (at 81.28 60.96) (diameter 0) (color 0 0 0 0)
+  )
   (junction (at 212.09 160.655) (diameter 0) (color 0 0 0 0)
   )
@@
     (stroke (width 0) (type default))
   )
+  (wire (pts (xy 81.28 60.96) (xy 100.33 60.96))
+    (stroke (width 0) (type default))
+  )
   (wire (pts (xy 240.03 215.9) (xy 240.03 234.315))
     (stroke (width 0) (type default))
@@
     (stroke (width 0) (type default))
   )
-  (wire (pts (xy 87.63 60.96) (xy 100.33 60.96))
+  (wire (pts (xy 77.47 60.96) (xy 81.28 60.96))
     (stroke (width 0) (type default))
   )
@@
     (stroke (width 0) (type default))
   )
-  (wire (pts (xy 81.28 35.56) (xy 81.28 48.26))
+  (wire (pts (xy 81.28 35.56) (xy 81.28 60.96))
     (stroke (width 0) (type default))
   )
@@
     (stroke (width 0) (type default))
   )
-  (wire (pts (xy 68.58 83.82) (xy 68.58 91.44))
-    (stroke (width 0) (type default))
-  )
   (wire (pts (xy 102.87 171.45) (xy 96.52 171.45))
     (stroke (width 0) (type default))
@@
     (stroke (width 0) (type default))
   )
+  (wire (pts (xy 88.9 83.82) (xy 100.33 83.82))
+    (stroke (width 0) (type default))
+  )
   (wire (pts (xy 267.97 271.145) (xy 240.03 271.145))
     (stroke (width 0) (type default))
@@
     (stroke (width 0) (type default))
   )
+  (wire (pts (xy 53.34 53.34) (xy 54.61 53.34))
+    (stroke (width 0) (type default))
+  )
   (wire (pts (xy 154.94 83.82) (xy 157.48 83.82))
     (stroke (width 0) (type default))
@@
     (stroke (width 0) (type default))
   )
+  (wire (pts (xy 67.31 50.8) (xy 100.33 50.8))
+    (stroke (width 0) (type default))
+  )
   (wire (pts (xy 212.09 133.35) (xy 212.09 134.62))
     (stroke (width 0) (type default))
@@
     (stroke (width 0) (type default))
   )
+  (wire (pts (xy 68.58 86.36) (xy 68.58 91.44))
+    (stroke (width 0) (type default))
+  )
   (wire (pts (xy 240.03 207.01) (xy 243.84 207.01))
     (stroke (width 0) (type default))
@@
     (stroke (width 0) (type default))
   )
-  (wire (pts (xy 68.58 83.82) (xy 100.33 83.82))
-    (stroke (width 0) (type default))
-  )
   (wire (pts (xy 186.055 174.625) (xy 186.055 183.515))
     (stroke (width 0) (type default))
@@
     (stroke (width 0) (type default))
   )
+  (wire (pts (xy 67.31 53.34) (xy 100.33 53.34))
+    (stroke (width 0) (type default))
+  )
   (wire (pts (xy 260.985 180.975) (xy 260.985 174.625))
     (stroke (width 0) (type default))
@@
     (stroke (width 0) (type default))
   )
-  (wire (pts (xy 88.9 86.36) (xy 100.33 86.36))
-    (stroke (width 0) (type default))
-  )
   (wire (pts (xy 243.84 174.625) (xy 241.935 174.625))
     (stroke (width 0) (type default))
@@
     (stroke (width 0) (type default))
   )
-  (wire (pts (xy 53.34 50.8) (xy 100.33 50.8))
-    (stroke (width 0) (type default))
-  )
   (wire (pts (xy 288.29 154.305) (xy 271.78 154.305))
     (stroke (width 0) (type default))
@@
     (stroke (width 0) (type default))
   )
-  (wire (pts (xy 81.28 48.26) (xy 91.44 48.26))
-    (stroke (width 0) (type default))
-  )
   (wire (pts (xy 260.985 174.625) (xy 259.08 174.625))
     (stroke (width 0) (type default))
@@
     (stroke (width 0) (type default))
   )
-  (wire (pts (xy 53.34 53.34) (xy 100.33 53.34))
-    (stroke (width 0) (type default))
-  )
   (wire (pts (xy 186.055 248.285) (xy 186.055 257.175))
     (stroke (width 0) (type default))
@@
     (stroke (width 0) (type default))
   )
-  (wire (pts (xy 88.9 86.36) (xy 88.9 91.44))
+  (wire (pts (xy 88.9 83.82) (xy 88.9 91.44))
     (stroke (width 0) (type default))
   )
@@
     (stroke (width 0) (type default))
   )
+  (wire (pts (xy 100.33 86.36) (xy 68.58 86.36))
+    (stroke (width 0) (type default))
+  )
   (wire (pts (xy 86.36 58.42) (xy 86.36 55.88))
     (stroke (width 0) (type default))
@@
     (stroke (width 0) (type default))
   )
+  (wire (pts (xy 53.34 50.8) (xy 54.61 50.8))
+    (stroke (width 0) (type default))
+  )
   (wire (pts (xy 267.97 234.315) (xy 240.03 234.315))
     (stroke (width 0) (type default))
@@
     (effects (font (size 1.27 1.27)) (justify left bottom))
   )
-  (label "row0" (at 157.48 53.34 0) (fields_autoplaced)
+  (label "row0" (at 157.48 66.04 0) (fields_autoplaced)
     (effects (font (size 1.27 1.27)) (justify left bottom))
   )
@@
     (effects (font (size 1.27 1.27)) (justify right bottom))
   )
-  (label "row2" (at 157.48 58.42 0) (fields_autoplaced)
+  (label "row2" (at 157.48 60.96 0) (fields_autoplaced)
     (effects (font (size 1.27 1.27)) (justify left bottom))
   )
@@
     (effects (font (size 1.27 1.27)) (justify left bottom))
   )
-  (label "row1" (at 157.48 55.88 0) (fields_autoplaced)
+  (label "row1" (at 157.48 63.5 0) (fields_autoplaced)
     (effects (font (size 1.27 1.27)) (justify left bottom))
   )
-  (label "rotA" (at 157.48 63.5 0) (fields_autoplaced)
+  (label "rotA" (at 157.48 55.88 0) (fields_autoplaced)
     (effects (font (size 1.27 1.27)) (justify left bottom))
   )
@@
     (effects (font (size 1.27 1.27)) (justify left bottom))
   )
-  (label "row3" (at 157.48 60.96 0) (fields_autoplaced)
+  (label "row3" (at 157.48 58.42 0) (fields_autoplaced)
     (effects (font (size 1.27 1.27)) (justify left bottom))
   )
-  (label "col2" (at 157.48 78.74 0) (fields_autoplaced)
+  (label "col2" (at 157.48 83.82 0) (fields_autoplaced)
     (effects (font (size 1.27 1.27)) (justify left bottom))
   )
@@
     (effects (font (size 1.27 1.27)) (justify right bottom))
   )
-  (label "col3" (at 157.48 76.2 0) (fields_autoplaced)
+  (label "col3" (at 157.48 86.36 0) (fields_autoplaced)
     (effects (font (size 1.27 1.27)) (justify left bottom))
   )
@@
     (effects (font (size 1.27 1.27)) (justify right bottom))
   )
-  (label "led0" (at 157.48 86.36 0) (fields_autoplaced)
+  (label "led0" (at 157.48 76.2 0) (fields_autoplaced)
     (effects (font (size 1.27 1.27)) (justify left bottom))
   )
-  (label "col0" (at 157.48 83.82 0) (fields_autoplaced)
+  (label "col0" (at 157.48 78.74 0) (fields_autoplaced)
     (effects (font (size 1.27 1.27)) (justify left bottom))
   )
-  (label "rotB" (at 157.48 66.04 0) (fields_autoplaced)
+  (label "rotB" (at 157.48 53.34 0) (fields_autoplaced)
     (effects (font (size 1.27 1.27)) (justify left bottom))
   )
@@
     )
   )
+  (symbol (lib_id "Device:R") (at 60.96 50.8 90) (unit 1)
+    (in_bom yes) (on_board yes) (dnp no) (fields_autoplaced)
+    (property "Reference" "R5" (at 57.15 50.8 90)
+      (effects (font (size 1.27 1.27)))
+    )
+    (property "Value" "22" (at 63.5 50.8 90)
+      (effects (font (size 1.27 1.27)))
+    )
+    (property "Footprint" "Resistor_THT:R_Axial_DIN0207_L6.3mm_D2.5mm_P7.62mm_Horizontal" (at 62.738 50.8 90)
+      (effects (font (size 1.27 1.27)) hide)
+    )
+    (property "Datasheet" "~" (at 60.96 50.8 0)
+      (effects (font (size 1.27 1.27)) hide)
+    )
+    (pin "1")
+    (pin "2")
+    (instances
+      (project "RB-Macro16"
+        (path "/9538e4ed-27e6-4c37-b989-9859dc0d49e8"
+          (reference "R5") (unit 1)
+        )
+      )
+    )
+  )
   (symbol (lib_id "Device:C_Small") (at 102.87 177.8 0) (unit 1)
     (in_bom yes) (on_board yes) (dnp no) (fields_autoplaced)
@@
     )
   )
+  (symbol (lib_id "Device:R") (at 60.96 53.34 90) (unit 1)
+    (in_bom yes) (on_board yes) (dnp no)
+    (property "Reference" "R6" (at 57.15 53.34 90)
+      (effects (font (size 1.27 1.27)))
+    )
+    (property "Value" "22" (at 63.5 53.34 90)
+      (effects (font (size 1.27 1.27)))
+    )
+    (property "Footprint" "Resistor_THT:R_Axial_DIN0207_L6.3mm_D2.5mm_P7.62mm_Horizontal" (at 62.738 53.34 90)
+      (effects (font (size 1.27 1.27)) hide)
+    )
+    (property "Datasheet" "~" (at 60.96 53.34 0)
+      (effects (font (size 1.27 1.27)) hide)
+    )
+    (pin "1")
+    (pin "2")
+    (instances
+      (project "RB-Macro16"
+        (path "/9538e4ed-27e6-4c37-b989-9859dc0d49e8"
+          (reference "R6") (unit 1)
+        )
+      )
+    )
+  )
   (symbol (lib_name "C_1") (lib_id "Device:C") (at 216.535 260.985 0) (unit 1)
     (in_bom yes) (on_board yes) (dnp no)
@@
     )
   )
-  (symbol (lib_name "VCC_3") (lib_id "power:VCC") (at 87.63 60.96 90) (unit 1)
-    (in_bom yes) (on_board yes) (dnp no) (fields_autoplaced)
-    (property "Reference" "#PWR0102" (at 87.63 64.77 0)
+  (symbol (lib_name "VCC_3") (lib_id "power:VCC") (at 77.47 60.96 90) (unit 1)
+    (in_bom yes) (on_board yes) (dnp no)
+    (property "Reference" "#PWR0102" (at 77.47 64.77 0)
       (effects (font (size 1.27 1.27)) hide)
     )
-    (property "Value" "VCC" (at 85.09 60.96 90)
+    (property "Value" "VCC" (at 74.93 60.96 90)
       (effects (font (size 1.27 1.27)) (justify left))
     )
-    (property "Footprint" "" (at 87.63 60.96 0)
+    (property "Footprint" "" (at 77.47 60.96 0)
       (effects (font (size 1.27 1.27)) hide)
     )
-    (property "Datasheet" "" (at 87.63 60.96 0)
+    (property "Datasheet" "" (at 77.47 60.96 0)
       (effects (font (size 1.27 1.27)) hide)
     )
